File: hw/forcegauge/forcegauge.sch (KiCad schematic (older format))
At the start: 6 parts

Commit message: schematic updated
Parts:
- added C?: 10uF, Capacitor_SMD:C_0603_1608Metric, symbol Device:C
- added C? (x2): 100nF, Capacitor_SMD:C_0603_1608Metric, symbol Device:C
- added C? (x2): 22uF, Capacitor_SMD:C_1812_4532Metric, symbol Device:C
- added D? (x2): LED, Diode_SMD:D_0603_1608Metric, symbol Device:LED
- added D?: D_Schottky, Diode_SMD:D_SMA, symbol Device:D_Schottky
- added D?: D, symbol Device:D
- added L?: 22uH, symbol Device:L
- added Q? (x4): FDS6892A, Package_SO:SOIC-8_3.9x4.9mm_P1.27mm, symbol Transistor_FET:FDS6892A
- added Q?: Q_PMOS_DGS, Package_TO_SOT_SMD:SOT-323_SC-70, symbol Device:Q_PMOS_DGS
- added R? (x2): 2k, Resistor_SMD:R_0603_1608Metric, symbol Device:R
- added R?: 100, Resistor_SMD:R_0603_1608Metric, symbol Device:R
- added R? (x3): 1k, Resistor_SMD:R_0603_1608Metric, symbol Device:R
- added R?: 7.5k, Resistor_SMD:R_0603_1608Metric, symbol Device:R
- added R? (x5): 100k, Resistor_SMD:R_0603_1608Metric, symbol Device:R
- added SW? (x3): SW_Push, Button_Switch_THT:SW_PUSH_6mm, symbol Switch:SW_Push
- U?: Alternative (none) -> http://hmsemi.com/downfile/DW01A.PDF
Connections:
- net GND: now reaches U?.1 (TEMP)
- net GND: now also J?.5 (GND), J?.6 (Shield), U?.2 (GND), U?.3 (GND), C?.2, C?.2, C?.2, C?.2, Q?.3 (S2), Q?.3 (S2), Q?.7 (D1), Q?.8 (D1), R?.1, R?.1, R?.1, R?.2, SW?.2
- net at U?.2 (PROG): now also R?.1
- net VBUS: now reaches U?.4 (VCC)
- net VBUS: now also J?.1 (VBUS), U?.8 (CE), C?.1, C?.1, R?.2, R?.2
- net VCC: now reaches U?.5 (BAT)
- net VCC: now also U?.5 (IN), C?.1, L?.1, Q?.3 (S), R?.1, R?.2, R?.2
- net at U?.6 (STDBY): now also D?.1 (K)
- net at U?.7 (CHRG): now also D?.1 (K)
- net D-: now reaches J?.2 (D-)
- net D+: now reaches J?.3 (D+)
- net at U?.1 (SW): now also D?.2 (A), L?.2
- net at U?.3 (FB): now also R?.1, R?.2
- net 5V_EN: now reaches U?.4 (EN)
- net 5V_EN: now also Q?.1 (D), R?.2
- net at U?.1 (OD): now also Q?.2 (G1)
- net at U?.2 (CS): now also R?.1
- net at U?.3 (OC): now also Q?.4 (G2)
- net at U?.5 (VCC): now also C?.1, R?.2
- net BAT-: now reaches U?.6 (GND)
- net BAT-: now also C?.2, Q?.1 (S1), R?.2
- new net: D?.2 (A), R?.1 (x2)
- new net: D?.1 (K), Q?.4 (G2), R?.1, SW?.1
- new net: C?.1, D?.1 (K), R?.2
- new net: Q?.5 (D2), Q?.6 (D2), Q?.7 (D1), Q?.8 (D1)
- new net: D?.2 (A), Q?.1 (S1), Q?.2 (G), R?.1
- new net +3V3: R?.2
- new net BTN_PWR: Q?.5 (D2), Q?.6 (D2), R?.1
- new net PWR_EN: Q?.2 (G1), R?.2
Other:
- note added: "Charging current:\n3k - 400mA\n2k - 580mA\n1.6k - 690mA"
- moved on the sheet: J?, U?

Commit message: added schematic
Parts:
- removed C?: 100nF, Capacitor_SMD:C_0603_1608Metric, symbol Device:C
- removed Q?: Q_PMOS_DGS, Package_TO_SOT_SMD:SOT-323_SC-70, symbol Device:Q_PMOS_DGS
- added C? (x7): 100nF, Capacitor_SMD:C_0603_1608Metric, symbol Device:C
- added C? (x4): 10uF, Capacitor_SMD:C_0603_1608Metric, symbol Device:C
- added J?: OLDED_Screen, symbol Connector_Generic:Conn_01x04
- added J?: Load Cell, symbol Connector_Generic:Conn_01x04
- added J?: Battery, symbol Connector_Generic:Conn_01x02
- added Q?: SM2331PSA P-MOSFET, Package_TO_SOT_SMD:SOT-23_Handsoldering, symbol Device:Q_PMOS_GSD
- added Q?: S8550, Package_TO_SOT_THT:TO-92_Inline, symbol Transistor_BJT:S8550
- added R? (x2): 0R, Resistor_SMD:R_0603_1608Metric, symbol Device:R
- added R? (x2): 1k, Resistor_SMD:R_0603_1608Metric, symbol Device:R
- added R?: 20k, Resistor_SMD:R_0603_1608Metric, symbol Device:R
- added R?: 8k2, Resistor_SMD:R_0603_1608Metric, symbol Device:R
- added R? (x2): 470R, Resistor_SMD:R_0603_1608Metric, symbol Device:R
- added R? (x5): 10k, Resistor_SMD:R_0603_1608Metric, symbol Device:R
- added R?: 390k, Resistor_SMD:R_0603_1608Metric, symbol Device:R
- added R?: 100k, Resistor_SMD:R_0603_1608Metric, symbol Device:R
- added U?: HX711, Package_SO:SOP-16_4.55x10.3mm_P1.27mm, symbol Symbols:HX711
- added U?: LM1117-3.3, symbol Regulator_Linear:LM1117-3.3
- gave numbers to parts that had none: 3
Connections:
- net BTN_PWR is gone; now on net BTN_2: Q?.5 (D2), Q?.6 (D2), R?.1
- net +3V3: now also U?.8 (VCC), C?.1, C?.1, C?.1, J?.2 (Pin_2), R?.1, R?.1, R?.1, R?.2, R?.2, U?.16 (DVDD), U?.2 (VO)
- net 5V_EN: now also Q?.3 (D)
- net BAT-: now also J?.2 (Pin_2)
- net D+: now also U?.1 (UD+)
- net D-: now also U?.2 (UD-)
- net GND: now also D?.1 (K), Q?.4 (G2), R?.1, SW1.2, SW2.1, SW3.2, U?.3 (GND), U?.9 (GND), C?.1, C?.2, C?.2, C?.2, C?.2, C?.2, C?.2, C?.2, J?.1 (Pin_1), R?.1, R?.2, R?.2, U?.1 (GND), U?.10 (INPB), U?.14 (XI), U?.9 (INNB); no longer Q?.3 (S2), Q?.7 (D1), Q?.8 (D1), R?.1, SW2.2
- net PWR_EN: now also U?.10 (GPIO15), R?.2
- net VBUS: now also U?.5 (VCC), C?.1
- net VCC: now also J?.1 (Pin_1), Q?.2 (S), R?.1
- net at U?.1 (REST): now also R?.2
- net BUZZER: now reaches U?.11 (GPIO2)
- net BTN_3: now reaches U?.12 (GPIO0)
- net BTN_3: now also SW3.1, R?.1
- net SDA: now reaches U?.13 (GPIO4)
- net SDA: now also J?.4 (Pin_4)
- net SCL: now reaches U?.14 (GPIO5)
- net SCL: now also J?.3 (Pin_3)
- net RXD: now reaches U?.15 (RXD)
- net RXD: now also R?.2
- net TXD: now reaches U?.16 (TXD)
- net TXD: now also R?.2
- net V_BAT: now reaches U?.2 (ADC)
- net V_BAT: now also C?.1, R?.1, R?.2
- net at U?.3 (CH_PD): now also R?.2
- net BTN_2: now reaches U?.4 (GPIO16)
- net DOUT: now reaches U?.5 (GPIO14)
- net DOUT: now also U?.12 (DOUT)
- net CLK: now reaches U?.6 (GPIO12)
- net CLK: now also U?.11 (PD_SCK)
- net BTN_1: now reaches U?.7 (GPIO13)
- net BTN_1: now also SW1.1, R?.2
- net at U?.6 (TXD): now also R?.1
- net at U?.7 (RXD): now also R?.1
- net at U?.8 (V3): now also C?.1
- net at U?.1 (OD): now also Q?.2 (G1)
- net +5V: now reaches C?.1, D?.1 (K), R?.2
- net +5V: now also C?.1, C?.2, Q?.1 (E), U?.1 (VSUP), U?.3 (VI)
- net at D?.2 (A), Q?.1 (S1), R?.1: now also Q?.1 (G)
- new net: Q?.3 (S2), Q?.7 (D1), Q?.8 (D1), R?.1, SW2.2
- new net: R?.1, U?.15 (RATE)
- new net: Q?.2 (B), U?.2 (BASE)
- new net: R?.1, R?.2, U?.4 (VFB)
- new net: C?.1, U?.6 (VBG)
- new net: C?.1, R?.2, U?.7 (INNA)
- new net: C?.2, R?.2, U?.8 (INPA)
- new net A+: J?.4 (Pin_4), R?.1
- new net A-: J?.3 (Pin_3), R?.1
- new net E+: C?.2, J?.1 (Pin_1), Q?.3 (C), R?.1, U?.3 (AVDD)
- new net E-: C?.1, C?.2, J?.2 (Pin_2), R?.1, R?.2, U?.5 (AGND)
Other:
- note added: "15/06/2021\n"
- note added: "A0 - A0\nD0 - GPIO 16\nD1 - GPIO 5\nD2 - GPIO 4\nD3 - GPIO 0\nD4 - GPIO 2\nD5 - GPIO 14\nD6 - GPIO 12\nD7 - GPIO 13\nD8 - GPIO 15\nSD2- GPIO 9\nSD3- GPIO 10\nRX - GPIO 3\nTX - GPIO 1"
- note added: "Force Gauge"
- note added: "v0.1"
- moved on the sheet: C?, D?, J?, L?, Q?A, Q?B, R?, SW1, SW2, SW3, U?
