File: hw/forcegauge/forcegauge.kicad_sch (KiCad schematic)
At the start: 69 parts, among them J1 USB_B_Micro, J2 Battery, J3 OLDED_Screen, J4 Conn_01x05, Q1 FDS6892A, Q2 BSS138, Q3 SM2331PSA P-MOSFET, Q4 S8550, Q5 FDS6892A, SW1 SW_Push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

Commit message: pcb WIP
Parts:
- gave numbers to parts that had none: 1
Connections:
- net GND: now also Q5.1 (S1), Q5.5 (D2), Q5.6 (D2), R28.1, SW2.2; no longer D4.1 (K), Q5.2 (G1), R15.1, SW2.1
- new net: D4.1 (K), Q5.2 (G1), R15.1, SW2.1
Changed lines of the file:
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@@
   (junction (at 182.88 149.86) (diameter 0) (color 0 0 0 0)
   )
-  (junction (at 171.45 163.83) (diameter 0) (color 0 0 0 0)
-  )
   (junction (at 33.02 96.52) (diameter 0) (color 0 0 0 0)
   )
@@
     (stroke (width 0) (type default) (color 0 0 0 0))
   )
+  (wire (pts (xy 223.52 167.64) (xy 223.52 163.83))
+    (stroke (width 0) (type default) (color 0 0 0 0))
+  )
   (wire (pts (xy 54.61 154.94) (xy 54.61 151.13))
     (stroke (width 0) (type default) (color 0 0 0 0))
@@
     (stroke (width 0) (type default) (color 0 0 0 0))
   )
-  (wire (pts (xy 171.45 165.1) (xy 171.45 163.83))
-    (stroke (width 0) (type default) (color 0 0 0 0))
-  )
   (wire (pts (xy 22.86 40.64) (xy 25.4 40.64))
     (stroke (width 0) (type default) (color 0 0 0 0))
@@
       (effects (font (size 1.27 1.27) italic) (justify left) hide)
     )
-    (property "Datasheet" "http://www.fairchildsemi.com/ds/FD/FDS6892A.pdf" (id 3) (at 220.98 156.21 0)
+    (property "Datasheet" "https://www.onsemi.com/pdf/datasheet/fds6892a-d.pdf" (id 3) (at 220.98 156.21 0)
       (effects (font (size 1.27 1.27)) (justify left) hide)
     )
@@
       (effects (font (size 1.27 1.27) italic) (justify left) hide)
     )
-    (property "Datasheet" "http://www.fairchildsemi.com/ds/FD/FDS6892A.pdf" (id 3) (at 251.46 156.21 0)
+    (property "Datasheet" "https://www.onsemi.com/pdf/datasheet/fds6892a-d.pdf" (id 3) (at 251.46 156.21 0)
       (effects (font (size 1.27 1.27)) (justify left) hide)
     )
@@
     (pin "6")
   )
-  (symbol (lib_id "power:GND") (at 171.45 165.1 0) (unit 1)
+  (symbol (lib_id "power:GND") (at 223.52 167.64 0) (unit 1)
     (in_bom yes) (on_board yes)
-    (property "Reference" "#PWR0113" (id 0) (at 171.45 171.45 0)
+    (property "Reference" "#PWR0113" (id 0) (at 223.52 173.99 0)
       (effects (font (size 1.27 1.27)) hide)
     )
-    (property "Value" "GND" (id 1) (at 171.577 169.4942 0))
-    (property "Footprint" "" (id 2) (at 171.45 165.1 0)
+    (property "Value" "GND" (id 1) (at 223.647 172.0342 0))
+    (property "Footprint" "" (id 2) (at 223.52 167.64 0)
       (effects (font (size 1.27 1.27)) hide)
     )
-    (property "Datasheet" "" (id 3) (at 171.45 165.1 0)
+    (property "Datasheet" "" (id 3) (at 223.52 167.64 0)
       (effects (font (size 1.27 1.27)) hide)
     )
@@
   (symbol (lib_id "power:GND") (at 267.97 93.98 0) (unit 1)
     (in_bom yes) (on_board yes)
-    (property "Reference" "#PWR?" (id 0) (at 267.97 100.33 0)
+    (property "Reference" "#PWR0139" (id 0) (at 267.97 100.33 0)
       (effects (font (size 1.27 1.27)) hide)
     )
@@
   (symbol (lib_id "Device:C") (at 267.97 88.9 0) (unit 1)
     (in_bom yes) (on_board yes)
-    (property "Reference" "C?" (id 0) (at 273.05 87.63 90)
+    (property "Reference" "C16" (id 0) (at 273.05 87.63 90)
       (effects (font (size 1.27 1.27)) (justify left))
     )
@@
     )
     (path "/1df6bffc-de61-4d01-87d9-16f350714abc"
-      (reference "#PWR?") (unit 1) (value "GND") (footprint "")
+      (reference "#PWR0139") (unit 1) (value "GND") (footprint "")
     )
     (path "/00000000-0000-0000-0000-000060d804d9"
@@
     )
     (path "/69652816-8db9-4b3d-af69-22d22f10ef32"
-      (reference "C?") (unit 1) (value "100nF") (footprint "Capacitor_SMD:C_0603_1608Metric")
+      (reference "C16") (unit 1) (value "100nF") (footprint "Capacitor_SMD:C_0603_1608Metric")
     )
     (path "/00000000-0000-0000-0000-000060b889ed"

Commit message: PCB wip
Changed lines of the file:
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@@
     (pin "15")
     (pin "16")
-    (pin "17")
-    (pin "18")
-    (pin "19")
     (pin "2")
-    (pin "20")
-    (pin "21")
-    (pin "22")
     (pin "3")
     (pin "4")

Commit message: pcb routing finished, todo check
Parts:
- added H1, H2, H3, H4: MountingHole, forcegauge:MountingHole_2mm_OLED, symbol Mechanical:MountingHole
Changed lines of the file:
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@@
     (pin "2")
+  )
+  (symbol (lib_id "Mechanical:MountingHole") (at 161.29 187.96 0) (unit 1)
+    (in_bom yes) (on_board yes) (fields_autoplaced)
+    (property "Reference" "H3" (id 0) (at 163.83 186.6899 0)
+      (effects (font (size 1.27 1.27)) (justify left))
+    )
+    (property "Value" "MountingHole" (id 1) (at 163.83 189.2299 0)
+      (effects (font (size 1.27 1.27)) (justify left))
+    )
+    (property "Footprint" "forcegauge:MountingHole_2mm_OLED" (id 2) (at 161.29 187.96 0)
+      (effects (font (size 1.27 1.27)) hide)
+    )
+    (property "Datasheet" "~" (id 3) (at 161.29 187.96 0)
+      (effects (font (size 1.27 1.27)) hide)
+    )
   )
   (symbol (lib_id "power:GND") (at 267.97 93.98 0) (unit 1)
@@
     (pin "2")
   )
+  (symbol (lib_id "Mechanical:MountingHole") (at 161.29 177.8 0) (unit 1)
+    (in_bom yes) (on_board yes) (fields_autoplaced)
+    (property "Reference" "H1" (id 0) (at 163.83 176.5299 0)
+      (effects (font (size 1.27 1.27)) (justify left))
+    )
+    (property "Value" "MountingHole" (id 1) (at 163.83 179.0699 0)
+      (effects (font (size 1.27 1.27)) (justify left))
+    )
+    (property "Footprint" "forcegauge:MountingHole_2mm_OLED" (id 2) (at 161.29 177.8 0)
+      (effects (font (size 1.27 1.27)) hide)
+    )
+    (property "Datasheet" "~" (id 3) (at 161.29 177.8 0)
+      (effects (font (size 1.27 1.27)) hide)
+    )
+  )
+  (symbol (lib_id "Mechanical:MountingHole") (at 161.29 193.04 0) (unit 1)
+    (in_bom yes) (on_board yes) (fields_autoplaced)
+    (property "Reference" "H4" (id 0) (at 163.83 191.7699 0)
+      (effects (font (size 1.27 1.27)) (justify left))
+    )
+    (property "Value" "MountingHole" (id 1) (at 163.83 194.3099 0)
+      (effects (font (size 1.27 1.27)) (justify left))
+    )
+    (property "Footprint" "forcegauge:MountingHole_2mm_OLED" (id 2) (at 161.29 193.04 0)
+      (effects (font (size 1.27 1.27)) hide)
+    )
+    (property "Datasheet" "~" (id 3) (at 161.29 193.04 0)
+      (effects (font (size 1.27 1.27)) hide)
+    )
+  )
+  (symbol (lib_id "Mechanical:MountingHole") (at 161.29 182.88 0) (unit 1)
+    (in_bom yes) (on_board yes) (fields_autoplaced)
+    (property "Reference" "H2" (id 0) (at 163.83 181.6099 0)
+      (effects (font (size 1.27 1.27)) (justify left))
+    )
+    (property "Value" "MountingHole" (id 1) (at 163.83 184.1499 0)
+      (effects (font (size 1.27 1.27)) (justify left))
+    )
+    (property "Footprint" "forcegauge:MountingHole_2mm_OLED" (id 2) (at 161.29 182.88 0)
+      (effects (font (size 1.27 1.27)) hide)
+    )
+    (property "Datasheet" "~" (id 3) (at 161.29 182.88 0)
+      (effects (font (size 1.27 1.27)) hide)
+    )
+  )
   (sheet_instances
     (path "/" (page "1"))
@@
       (reference "D4") (unit 1) (value "1SS355") (footprint "Diode_SMD:D_SOD-323_HandSoldering")
     )
+    (path "/7c02e4ac-b219-4394-88fd-5f1bff0e4084"
+      (reference "H1") (unit 1) (value "MountingHole") (footprint "forcegauge:MountingHole_2mm_OLED")
+    )
+    (path "/d10c5232-4237-4c2a-895a-1f55828f1482"
+      (reference "H2") (unit 1) (value "MountingHole") (footprint "forcegauge:MountingHole_2mm_OLED")
+    )
+    (path "/06152ca9-8688-42fa-a575-8f095f3837e1"
+      (reference "H3") (unit 1) (value "MountingHole") (footprint "forcegauge:MountingHole_2mm_OLED")
+    )
+    (path "/98c061e6-bc83-426a-99cb-a9b9832a9118"
+      (reference "H4") (unit 1) (value "MountingHole") (footprint "forcegauge:MountingHole_2mm_OLED")
+    )
     (path "/00000000-0000-0000-0000-000060a428c7"

Commit message: pcb v0.1 sent
Parts:
- D2: value LED -> LED RED
- D3: value LED -> LED GREEN
- J4: value Conn_01x05 -> Load Cell
Connections:
- net BAT-: no longer R2.2
- net GND: now also R2.2
Changed lines of the file:
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@@
   (junction (at 93.98 26.67) (diameter 0) (color 0 0 0 0)
   )
+  (junction (at 71.12 133.35) (diameter 0) (color 0 0 0 0)
+  )
   (junction (at 189.23 46.99) (diameter 0) (color 0 0 0 0)
   )
@@
   (junction (at 212.09 113.03) (diameter 0) (color 0 0 0 0)
   )
-  (junction (at 71.12 133.35) (diameter 0) (color 0 0 0 0)
+  (junction (at 31.75 143.51) (diameter 0) (color 0 0 0 0)
   )
   (junction (at 105.41 130.81) (diameter 0) (color 0 0 0 0)
@@
     (stroke (width 0) (type default) (color 0 0 0 0))
   )
-  (wire (pts (xy 59.69 143.51) (xy 76.2 143.51))
+  (wire (pts (xy 59.69 143.51) (xy 71.12 143.51))
     (stroke (width 0) (type default) (color 0 0 0 0))
   )
@@
     (stroke (width 0) (type default) (color 0 0 0 0))
   )
-  (wire (pts (xy 27.94 124.46) (xy 27.94 133.35))
-    (stroke (width 0) (type default) (color 0 0 0 0))
-  )
   (wire (pts (xy 199.39 91.44) (xy 199.39 92.71))
     (stroke (width 0) (type default) (color 0 0 0 0))
@@
     (stroke (width 0) (type default) (color 0 0 0 0))
   )
-  (wire (pts (xy 76.2 143.51) (xy 76.2 133.35))
+  (wire (pts (xy 71.12 143.51) (xy 71.12 133.35))
     (stroke (width 0) (type default) (color 0 0 0 0))
   )
@@
     (stroke (width 0) (type default) (color 0 0 0 0))
   )
+  (wire (pts (xy 27.94 143.51) (xy 31.75 143.51))
+    (stroke (width 0) (type default) (color 0 0 0 0))
+  )
   (wire (pts (xy 33.02 86.36) (xy 33.02 83.82))
     (stroke (width 0) (type default) (color 0 0 0 0))
@@
     (stroke (width 0) (type default) (color 0 0 0 0))
   )
+  (wire (pts (xy 27.94 124.46) (xy 27.94 143.51))
+    (stroke (width 0) (type default) (color 0 0 0 0))
+  )
   (wire (pts (xy 118.11 34.29) (xy 114.3 34.29))
     (stroke (width 0) (type default) (color 0 0 0 0))
@@
     (stroke (width 0) (type default) (color 0 0 0 0))
   )
-  (wire (pts (xy 27.94 133.35) (xy 71.12 133.35))
-    (stroke (width 0) (type default) (color 0 0 0 0))
-  )
   (wire (pts (xy 189.23 41.91) (xy 191.77 41.91))
     (stroke (width 0) (type default) (color 0 0 0 0))
@@
   (symbol (lib_id "Device:LED") (at 97.79 175.26 90) (unit 1)
     (in_bom yes) (on_board yes)
-    (property "Reference" "D2" (id 0) (at 100.7618 174.2694 90)
+    (property "Reference" "D2" (id 0) (at 93.345 175.26 90)
       (effects (font (size 1.27 1.27)) (justify right))
     )
-    (property "Value" "LED" (id 1) (at 100.7618 176.5808 90)
+    (property "Value" "LED RED" (id 1) (at 88.9 177.8 90)
       (effects (font (size 1.27 1.27)) (justify right))
     )
@@
       (effects (font (size 1.27 1.27)) (justify right))
     )
-    (property "Value" "LED" (id 1) (at 108.3818 176.5808 90)
+    (property "Value" "LED GREEN" (id 1) (at 107.95 176.53 90)
       (effects (font (size 1.27 1.27)) (justify right))
     )
@@
     (in_bom yes) (on_board yes)
     (property "Reference" "J4" (id 0) (at 165.9128 87.1982 0))
-    (property "Value" "Conn_01x05" (id 1) (at 165.9128 89.5096 0))
+    (property "Value" "Load Cell" (id 1) (at 165.9128 89.5096 0))
     (property "Footprint" "Connector_PinSocket_2.54mm:PinSocket_1x05_P2.54mm_Vertical" (id 2) (at 163.83 97.79 0)
       (effects (font (size 1.27 1.27)) hide)
@@
     )
     (path "/00000000-0000-0000-0000-000060b3a478"
-      (reference "D2") (unit 1) (value "LED") (footprint "Diode_SMD:D_0603_1608Metric")
+      (reference "D2") (unit 1) (value "LED RED") (footprint "Diode_SMD:D_0603_1608Metric")
     )
     (path "/00000000-0000-0000-0000-000060b46e0c"
-      (reference "D3") (unit 1) (value "LED") (footprint "Diode_SMD:D_0603_1608Metric")
+      (reference "D3") (unit 1) (value "LED GREEN") (footprint "Diode_SMD:D_0603_1608Metric")
     )
     (path "/00000000-0000-0000-0000-000060bfc449"
@@
     )
     (path "/00000000-0000-0000-0000-000060e7dc22"
-      (reference "J4") (unit 1) (value "Conn_01x05") (footprint "Connector_PinSocket_2.54mm:PinSocket_1x05_P2.54mm_Vertical")
+      (reference "J4") (unit 1) (value "Load Cell") (footprint "Connector_PinSocket_2.54mm:PinSocket_1x05_P2.54mm_Vertical")
     )
     (path "/00000000-0000-0000-0000-000060b88038"
