File: hw/forcegauge/forcegauge.kicad_sch (KiCad schematic)
At the start: 73 parts, among them J1 USB_B_Micro, J2 Battery, J3 OLDED_Screen, J4 Load Cell, Q1 FDS6892A, Q2 BSS138, Q3 SM2331PSA P-MOSFET, Q4 S8550, Q5 BSS138, SW1 SW_Push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

Commit message: pcb and box updata
Parts:
- added H? (x4): PCB Mounting hole, forcegauge:MountingHole_2mm_OLED, symbol Mechanical:MountingHole
Other:
- moved on the sheet: H1, H2, H3, H4
Changed lines of the file:
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@@
     (pin "3")
   )
-  (symbol (lib_id "Mechanical:MountingHole") (at 161.29 187.96 0) (unit 1)
+  (symbol (lib_id "Mechanical:MountingHole") (at 140.716 27.686 0) (unit 1)
+    (in_bom yes) (on_board yes)
+    (property "Reference" "H?" (id 0) (at 143.51 26.4159 0)
+      (effects (font (size 1.27 1.27)) (justify left))
+    )
+    (property "Value" "PCB Mounting hole" (id 1) (at 143.51 28.9559 0)
+      (effects (font (size 1.27 1.27)) (justify left))
+    )
+    (property "Footprint" "forcegauge:MountingHole_2mm_OLED" (id 2) (at 140.716 27.686 0)
+      (effects (font (size 1.27 1.27)) hide)
+    )
+    (property "Datasheet" "~" (id 3) (at 140.716 27.686 0)
+      (effects (font (size 1.27 1.27)) hide)
+    )
+  )
+  (symbol (lib_id "Mechanical:MountingHole") (at 161.29 188.468 0) (unit 1)
     (in_bom yes) (on_board yes) (fields_autoplaced)
-    (property "Reference" "H3" (id 0) (at 163.83 186.6899 0)
-      (effects (font (size 1.27 1.27)) (justify left))
-    )
-    (property "Value" "MountingHole" (id 1) (at 163.83 189.2299 0)
-      (effects (font (size 1.27 1.27)) (justify left))
-    )
-    (property "Footprint" "forcegauge:MountingHole_2mm_OLED" (id 2) (at 161.29 187.96 0)
-      (effects (font (size 1.27 1.27)) hide)
-    )
-    (property "Datasheet" "~" (id 3) (at 161.29 187.96 0)
+    (property "Reference" "H3" (id 0) (at 163.83 187.1979 0)
+      (effects (font (size 1.27 1.27)) (justify left))
+    )
+    (property "Value" "MountingHole" (id 1) (at 163.83 189.7379 0)
+      (effects (font (size 1.27 1.27)) (justify left))
+    )
+    (property "Footprint" "forcegauge:MountingHole_2mm_OLED" (id 2) (at 161.29 188.468 0)
+      (effects (font (size 1.27 1.27)) hide)
+    )
+    (property "Datasheet" "~" (id 3) (at 161.29 188.468 0)
       (effects (font (size 1.27 1.27)) hide)
     )
@@
     (pin "1")
     (pin "2")
+  )
+  (symbol (lib_id "Mechanical:MountingHole") (at 140.716 22.606 0) (unit 1)
+    (in_bom yes) (on_board yes)
+    (property "Reference" "H?" (id 0) (at 143.51 21.3359 0)
+      (effects (font (size 1.27 1.27)) (justify left))
+    )
+    (property "Value" "PCB Mounting hole" (id 1) (at 143.51 23.8759 0)
+      (effects (font (size 1.27 1.27)) (justify left))
+    )
+    (property "Footprint" "forcegauge:MountingHole_2mm_OLED" (id 2) (at 140.716 22.606 0)
+      (effects (font (size 1.27 1.27)) hide)
+    )
+    (property "Datasheet" "~" (id 3) (at 140.716 22.606 0)
+      (effects (font (size 1.27 1.27)) hide)
+    )
   )
   (symbol (lib_id "Device:Q_PNP_BEC") (at 201.93 77.47 180) (unit 1)
@@
     (pin "2")
   )
-  (symbol (lib_id "Mechanical:MountingHole") (at 161.29 177.8 0) (unit 1)
+  (symbol (lib_id "Mechanical:MountingHole") (at 161.29 178.308 0) (unit 1)
     (in_bom yes) (on_board yes) (fields_autoplaced)
-    (property "Reference" "H1" (id 0) (at 163.83 176.5299 0)
-      (effects (font (size 1.27 1.27)) (justify left))
-    )
-    (property "Value" "MountingHole" (id 1) (at 163.83 179.0699 0)
-      (effects (font (size 1.27 1.27)) (justify left))
-    )
-    (property "Footprint" "forcegauge:MountingHole_2mm_OLED" (id 2) (at 161.29 177.8 0)
-      (effects (font (size 1.27 1.27)) hide)
-    )
-    (property "Datasheet" "~" (id 3) (at 161.29 177.8 0)
-      (effects (font (size 1.27 1.27)) hide)
-    )
-  )
-  (symbol (lib_id "Mechanical:MountingHole") (at 161.29 193.04 0) (unit 1)
+    (property "Reference" "H1" (id 0) (at 163.83 177.0379 0)
+      (effects (font (size 1.27 1.27)) (justify left))
+    )
+    (property "Value" "MountingHole" (id 1) (at 163.83 179.5779 0)
+      (effects (font (size 1.27 1.27)) (justify left))
+    )
+    (property "Footprint" "forcegauge:MountingHole_2mm_OLED" (id 2) (at 161.29 178.308 0)
+      (effects (font (size 1.27 1.27)) hide)
+    )
+    (property "Datasheet" "~" (id 3) (at 161.29 178.308 0)
+      (effects (font (size 1.27 1.27)) hide)
+    )
+  )
+  (symbol (lib_id "Mechanical:MountingHole") (at 161.29 193.548 0) (unit 1)
     (in_bom yes) (on_board yes) (fields_autoplaced)
-    (property "Reference" "H4" (id 0) (at 163.83 191.7699 0)
-      (effects (font (size 1.27 1.27)) (justify left))
-    )
-    (property "Value" "MountingHole" (id 1) (at 163.83 194.3099 0)
-      (effects (font (size 1.27 1.27)) (justify left))
-    )
-    (property "Footprint" "forcegauge:MountingHole_2mm_OLED" (id 2) (at 161.29 193.04 0)
-      (effects (font (size 1.27 1.27)) hide)
-    )
-    (property "Datasheet" "~" (id 3) (at 161.29 193.04 0)
-      (effects (font (size 1.27 1.27)) hide)
-    )
-  )
-  (symbol (lib_id "Mechanical:MountingHole") (at 161.29 182.88 0) (unit 1)
+    (property "Reference" "H4" (id 0) (at 163.83 192.2779 0)
+      (effects (font (size 1.27 1.27)) (justify left))
+    )
+    (property "Value" "MountingHole" (id 1) (at 163.83 194.8179 0)
+      (effects (font (size 1.27 1.27)) (justify left))
+    )
+    (property "Footprint" "forcegauge:MountingHole_2mm_OLED" (id 2) (at 161.29 193.548 0)
+      (effects (font (size 1.27 1.27)) hide)
+    )
+    (property "Datasheet" "~" (id 3) (at 161.29 193.548 0)
+      (effects (font (size 1.27 1.27)) hide)
+    )
+  )
+  (symbol (lib_id "Mechanical:MountingHole") (at 140.716 37.846 0) (unit 1)
+    (in_bom yes) (on_board yes)
+    (property "Reference" "H?" (id 0) (at 143.51 36.5759 0)
+      (effects (font (size 1.27 1.27)) (justify left))
+    )
+    (property "Value" "PCB Mounting hole" (id 1) (at 143.51 39.1159 0)
+      (effects (font (size 1.27 1.27)) (justify left))
+    )
+    (property "Footprint" "forcegauge:MountingHole_2mm_OLED" (id 2) (at 140.716 37.846 0)
+      (effects (font (size 1.27 1.27)) hide)
+    )
+    (property "Datasheet" "~" (id 3) (at 140.716 37.846 0)
+      (effects (font (size 1.27 1.27)) hide)
+    )
+  )
+  (symbol (lib_id "Mechanical:MountingHole") (at 161.29 183.388 0) (unit 1)
     (in_bom yes) (on_board yes) (fields_autoplaced)
-    (property "Reference" "H2" (id 0) (at 163.83 181.6099 0)
-      (effects (font (size 1.27 1.27)) (justify left))
-    )
-    (property "Value" "MountingHole" (id 1) (at 163.83 184.1499 0)
-      (effects (font (size 1.27 1.27)) (justify left))
-    )
-    (property "Footprint" "forcegauge:MountingHole_2mm_OLED" (id 2) (at 161.29 182.88 0)
-      (effects (font (size 1.27 1.27)) hide)
-    )
-    (property "Datasheet" "~" (id 3) (at 161.29 182.88 0)
+    (property "Reference" "H2" (id 0) (at 163.83 182.1179 0)
+      (effects (font (size 1.27 1.27)) (justify left))
+    )
+    (property "Value" "MountingHole" (id 1) (at 163.83 184.6579 0)
+      (effects (font (size 1.27 1.27)) (justify left))
+    )
+    (property "Footprint" "forcegauge:MountingHole_2mm_OLED" (id 2) (at 161.29 183.388 0)
+      (effects (font (size 1.27 1.27)) hide)
+    )
+    (property "Datasheet" "~" (id 3) (at 161.29 183.388 0)
       (effects (font (size 1.27 1.27)) hide)
     )
@@
     )
     (pin "1")
+  )
+  (symbol (lib_id "Mechanical:MountingHole") (at 140.716 32.766 0) (unit 1)
+    (in_bom yes) (on_board yes)
+    (property "Reference" "H?" (id 0) (at 143.51 31.4959 0)
+      (effects (font (size 1.27 1.27)) (justify left))
+    )
+    (property "Value" "PCB Mounting hole" (id 1) (at 143.51 34.0359 0)
+      (effects (font (size 1.27 1.27)) (justify left))
+    )
+    (property "Footprint" "forcegauge:MountingHole_2mm_OLED" (id 2) (at 140.716 32.766 0)
+      (effects (font (size 1.27 1.27)) hide)
+    )
+    (property "Datasheet" "~" (id 3) (at 140.716 32.766 0)
+      (effects (font (size 1.27 1.27)) hide)
+    )
   )
   (sheet_instances
@@
       (reference "H4") (unit 1) (value "MountingHole") (footprint "forcegauge:MountingHole_2mm_OLED")
     )
+    (path "/052b7aad-f8b5-4b99-a424-4ddfe2a3337a"
+      (reference "H?") (unit 1) (value "PCB Mounting hole") (footprint "forcegauge:MountingHole_2mm_OLED")
+    )
+    (path "/6f142d01-9478-4cab-933a-944f5ce86a1d"
+      (reference "H?") (unit 1) (value "PCB Mounting hole") (footprint "forcegauge:MountingHole_2mm_OLED")
+    )
+    (path "/b3de04ae-2007-4a6d-8e48-724f8f2109eb"
+      (reference "H?") (unit 1) (value "PCB Mounting hole") (footprint "forcegauge:MountingHole_2mm_OLED")
+    )
+    (path "/fc828bf8-19a8-4e46-851c-671c99629a3a"
+      (reference "H?") (unit 1) (value "PCB Mounting hole") (footprint "forcegauge:MountingHole_2mm_OLED")
+    )
     (path "/00000000-0000-0000-0000-000060a428c7"

Commit message: v0.3 pcb
Parts:
- gave numbers to parts that had none: 4
Connections:
- net BTN_1: now also U6.11 (GPIO2); no longer U6.7 (GPIO13)
- net CLK: now also U6.5 (GPIO14); no longer U6.6 (GPIO12)
- net DOUT: now also U6.6 (GPIO12); no longer U6.5 (GPIO14)
- net PWR_EN: now also U6.7 (GPIO13); no longer U6.11 (GPIO2)
Other:
- moved on the sheet: R16, R25
